File: memory.kicad_sch (KiCad schematic)
At the start: 3 parts

Commit message: layout
Parts:
- R10, R9: renamed from R?; footprint (none) -> Resistor_SMD:R_0805_2012Metric
- gave numbers to parts that had none: 1
Changed lines of the file:
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@@
 		(on_board yes)
 		(dnp no)
-		(property "Reference" "#PWR?"
+		(property "Reference" "#PWR0103"
 			(at 182.88 90.17 0)
 			(effects
@@
 			(project "senior_design"
 				(path "/35c074f0-8545-4dc1-a57d-3ef0bc7d9188/97e7f441-78af-47c4-8e49-e87c6db6b63d"
-					(reference "#PWR?")
+					(reference "#PWR0103")
 					(unit 1)
 				)
@@
 		(on_board yes)
 		(dnp no)
-		(property "Reference" "R?"
+		(property "Reference" "R9"
 			(at 165.862 89.916 0)
 			(effects
@@
 			)
 		)
-		(property "Footprint" ""
+		(property "Footprint" "Resistor_SMD:R_0805_2012Metric"
 			(at 164.846 91.694 90)
 			(effects
@@
 			(project "senior_design"
 				(path "/35c074f0-8545-4dc1-a57d-3ef0bc7d9188/97e7f441-78af-47c4-8e49-e87c6db6b63d"
-					(reference "R?")
+					(reference "R9")
 					(unit 1)
 				)
@@
 		(dnp no)
 		(fields_autoplaced yes)
-		(property "Reference" "U?"
+		(property "Reference" "U5"
 			(at 143.51 82.55 0)
 			(effects
@@
 			(project "senior_design"
 				(path "/35c074f0-8545-4dc1-a57d-3ef0bc7d9188/97e7f441-78af-47c4-8e49-e87c6db6b63d"
-					(reference "U?")
+					(reference "U5")
 					(unit 1)
 				)
@@
 		(dnp no)
 		(fields_autoplaced yes)
-		(property "Reference" "#PWR?"
+		(property "Reference" "#PWR0101"
 			(at 162.56 121.92 0)
 			(effects
@@
 			(project "senior_design"
 				(path "/35c074f0-8545-4dc1-a57d-3ef0bc7d9188/97e7f441-78af-47c4-8e49-e87c6db6b63d"
-					(reference "#PWR?")
+					(reference "#PWR0101")
 					(unit 1)
 				)
@@
 		(on_board yes)
 		(dnp no)
-		(property "Reference" "R?"
+		(property "Reference" "R10"
 			(at 184.658 92.71 0)
 			(effects
@@
 			)
 		)
-		(property "Footprint" ""
+		(property "Footprint" "Resistor_SMD:R_0805_2012Metric"
 			(at 183.896 94.234 90)
 			(effects
@@
 			(project "senior_design"
 				(path "/35c074f0-8545-4dc1-a57d-3ef0bc7d9188/97e7f441-78af-47c4-8e49-e87c6db6b63d"
-					(reference "R?")
+					(reference "R10")
 					(unit 1)
 				)
@@
 		(on_board yes)
 		(dnp no)
-		(property "Reference" "#PWR?"
+		(property "Reference" "#PWR0102"
 			(at 114.3 116.84 0)
 			(effects
@@
 			(project "senior_design"
 				(path "/35c074f0-8545-4dc1-a57d-3ef0bc7d9188/97e7f441-78af-47c4-8e49-e87c6db6b63d"
-					(reference "#PWR?")
-					(unit 1)
-				)
+					(reference "#PWR0102")
+					(unit 1)
+				)
