File: peripherals.kicad_sch (KiCad schematic)
At the start: 0 parts

Commit message: start of display
Parts:
- added C13: 10uF, symbol Device:C
- added C14, C15: 1uF, symbol Device:C
- added C16: 0.1uF, symbol Device:C
- added D3: MBR0540, Diode_SMD:D_SOD-123, symbol Diode:MBR0540
- added D4, D5: 1N4148, Diode_THT:D_DO-35_SOD27_P7.62mm_Horizontal, symbol Diode:1N4148
- added JP1, JP2: SolderJumper_2_Open, symbol Jumper:SolderJumper_2_Open
- added L1: 6.8uH, symbol Device:L
- added R13: 10k, symbol Device:R
- added R14, R15, R16: R, symbol Device:R
- added U1: TPS61169DCKR, TPS61169DCKR:SOT65P210X110-5N, symbol TPS61169DCKR:TPS61169DCKR
- added U3: RA8875L3N, RA8875L3N:QFP50P1600X1600X160-100N, symbol RA8875L3N:RA8875L3N
Connections:
- new net: C16.1, R14.2, R15.1, R16.1, U1.3 (FB)
- new net: JP1.2 (B), R14.1
- new net: JP2.2 (B), R16.2
- new net: D3.2 (A), L1.2, U1.1 (SW)
- new net: D4.2 (A), D5.2 (A), R13.2, U1.4 (CTRL)
- new net +24V: C14.1, C15.1, D3.1 (K)
- new net +5V: C13.1, L1.1, R13.1, U1.5 (VIN)
- new net Backlite: D5.1 (K)
- new net CORE_VDD: U3.17 (CORE_VDD), U3.38 (CORE_VDD), U3.86 (CORE_VDD)
- new net GND: C13.2, C14.2, C15.2, C16.2, JP1.1 (A), JP2.1 (A), R15.2, U1.2 (GND), U3.16 (GND), U3.26 (GND), U3.39 (GND), U3.85 (GND)
- new net PWM0: D4.1 (K)
- new net VDDP: U3.13 (VDDP), U3.40 (VDDP), U3.62 (VDDP), U3.87 (VDDP)

Commit message: schematic update
Parts:
- added C18, C23, C24, C25, C26: 0.1uF, symbol Device:C
- added C21, C22: 15pF, symbol Device:C
- added J5: Out_to_display, symbol Connector:Conn_01x40_Pin
- added J6: MCU_In, symbol Connector:Conn_01x08_Pin
- added R17, R18, R19, R20, R21, R22, R23, R24, R25, R26, R27, R28, R29, R30, R31, R32, R33, R34, R35, R36: 33, symbol Device:R
- added R37: 10k, symbol Device:R
- added R38: R, symbol Device:R
- added U7: 74HC4050D, 74HC4050D:SO16, symbol 74HC4050D:74HC4050D
- added Y1: 20MHz, symbol Device:Crystal
- U1: value TPS61169DCKR -> Boost Converter - TPS61169DCKR
Connections:
- net CORE_VDD is gone; now on net +1V5: U3.17 (CORE_VDD), U3.38 (CORE_VDD), U3.86 (CORE_VDD)
- net VDDP is gone; now on net +3.3V: U3.13 (VDDP), U3.40 (VDDP), U3.62 (VDDP), U3.87 (VDDP)
- net +24V: now also J5.2 (Pin_2)
- net GND: now also U3.1 (OSC_GNDP), U3.10 (TEST0), U3.11 (TEST1), U3.12 (TEST2), U3.23 (IICA0), U3.24 (IICA1), U3.28 (SIFS0), U3.33 (KIN4/GPI4), U3.34 (KIN3/GPI3), U3.35 (KIN2/GPI2), U3.36 (KIN1/GPI1), U3.37 (KIN0/GPI0), U3.45 (GPIX), U3.6 (OSC_GND), U3.61 (LDO_GND), U3.70 (ADC_GND), U3.81 (C86), C18.2, C21.1, C22.1, C23.2, C24.2, C25.2, C26.2, J5.13 (Pin_13), J5.14 (Pin_14), J5.21 (Pin_21), J5.22 (Pin_22), J5.23 (Pin_23), J5.29 (Pin_29), J5.3 (Pin_3), J5.36 (Pin_36), J5.5 (Pin_5), J5.6 (Pin_6), J5.7 (Pin_7), U7.8 (GND)
- net PWM0: now also U3.14 (PWM1)
- net LEDK: now reaches C16.1, R14.2, R15.1, R16.1, U1.3 (FB)
- net LEDK: now also J5.1 (Pin_1)
- net +3.3V: now reaches U3.2 (OSC_VDDP)
- net +3.3V: now also U3.25 (PS), U3.27 (SIFS1), U3.76 (ADC_VDD), U3.77 (~{RD}/EN), U3.78 (~{WR}/~{RW}), U3.79 (~{CS}), U3.80 (RS), R37.2, U7.1 (VCC)
- net X_1: now reaches U3.3 (XI)
- net X_1: now also C21.2, R38.1, Y1.2
- net X_0: now reaches U3.4 (XO)
- net X_0: now also C22.2, R38.2, Y1.1
- net SPI_CS_3V: now reaches U3.41 (~{SCS})
- net SPI_CS_3V: now also U7.6 (3Y)
- net RA_MISO: now reaches U3.42 (SDO)
- net MOSI_3V: now reaches U3.43 (SDI)
- net MOSI_3V: now also U7.4 (2Y)
- net SPI_CLK_3V: now reaches U3.44 (SCL)
- net SPI_CLK_3V: now also U7.2 (1Y)
- net ON/OFF: now reaches U3.46 (GPOX)
- net ON/OFF: now also J5.31 (Pin_31)
- net at U3.47 (HSYNC): now also R33.1
- net at U3.48 (VSYNC): now also R34.1
- net at U3.49 (PCLK): now also R35.1
- net +1V5: now reaches U3.5 (OSC_VDD)
- net +1V5: now also U3.60 (LDO_OUT), C23.1, C24.1, C25.1, C26.1
- net at U3.50 (DE): now also R36.1
- net at U3.51 (PDAT0): now also R17.1
- net at U3.52 (PDAT1): now also R20.1
- net at U3.53 (PDAT2): now also R18.1
- net at U3.54 (PDAT3): now also R19.1
- net at U3.55 (PDAT4): now also R21.1
- net at U3.56 (PDAT5): now also R22.1
- net at U3.57 (PDAT6): now also R23.1
- net at U3.58 (PDAT7): now also R24.1
- net at U3.59 (PDAT8): now also R25.1
- net at U3.63 (PDAT9): now also R26.1
- net at U3.64 (PDAT10): now also R27.1
- net at U3.65 (PDAT11): now also R28.1
- net at U3.66 (PDAT12): now also R29.1
- net at U3.67 (PDAT13): now also R30.1
- net at U3.68 (PDAT14): now also R31.1
- net at U3.69 (PDAT15): now also R32.1
- net WAIT: now reaches U3.7 (~{WAIT})
- net WAIT: now also J6.7 (Pin_7)
- net at U3.71 (ADC_VREF): now also C18.1
- net X-: now reaches U3.72 (XN)
- net X-: now also J5.39 (Pin_39)
- net Y+: now reaches U3.73 (YP)
- net Y+: now also J5.38 (Pin_38)
- net Y-: now reaches U3.74 (YN)
- net Y-: now also J5.40 (Pin_40)
- net X+: now reaches U3.75 (XP)
- net X+: now also J5.37 (Pin_37)
- net INT: now reaches U3.8 (~{INT})
- net INT: now also J6.8 (Pin_8)
- net at U3.9 (~{RST}): now also U7.10 (4Y)
- new net +3V3: J5.4 (Pin_4)
- new net B3: J5.24 (Pin_24), R17.2
- new net B4: J5.25 (Pin_25), R20.2
- new net B5: J5.26 (Pin_26), R18.2
- new net B6: J5.27 (Pin_27), R19.2
- new net B7: J5.28 (Pin_28), R21.2
- new net BACKLITE: J6.1 (Pin_1)
- new net CS: J6.5 (Pin_5), U7.7 (3A)
- new net DE: J5.34 (Pin_34), R36.2
- new net G2: J5.15 (Pin_15), R22.2
- new net G3: J5.16 (Pin_16), R23.2
- new net G4: J5.17 (Pin_17), R24.2
- new net G5: J5.18 (Pin_18), R25.2
- new net G6: J5.19 (Pin_19), R26.2
- new net G7: J5.20 (Pin_20), R27.2
- new net HSYNC: J5.32 (Pin_32), R33.2
- new net MISO: J6.3 (Pin_3)
- new net MOSI: J6.4 (Pin_4), U7.5 (2A)
- new net PCLK: R35.2
- new net PIXCLK: J5.30 (Pin_30)
- new net R3: J5.8 (Pin_8), R28.2
- new net R4: J5.9 (Pin_9), R29.2
- new net R5: J5.10 (Pin_10), R30.2
- new net R6: J5.11 (Pin_11), R31.2
- new net R7: J5.12 (Pin_12), R32.2
- new net RESET: J6.6 (Pin_6), R37.1, U7.9 (4A)
- new net SCK: J6.2 (Pin_2), U7.3 (1A)
- new net VSYNC: J5.33 (Pin_33), R34.2
Other:
- moved on the sheet: U3

Commit message: schematic finish
Parts:
- removed C13: 10uF, symbol Device:C
- removed D3: MBR0540, Diode_SMD:D_SOD-123, symbol Diode:MBR0540
- removed D4: 1N4148, Diode_THT:D_DO-35_SOD27_P7.62mm_Horizontal, symbol Diode:1N4148
- removed J6: MCU_In, symbol Connector:Conn_01x08_Pin
- removed JP1, JP2: SolderJumper_2_Open, symbol Jumper:SolderJumper_2_Open
- removed R13: 10k, symbol Device:R
- removed R14, R15, R16: R, symbol Device:R
- added C27: 1uF, Capacitor_SMD:C_0805_2012Metric, symbol Device:C
- added C28, C29, C30: 0.1uF, Capacitor_SMD:C_0805_2012Metric, symbol Device:C
- added C31: .01uF, Capacitor_SMD:C_0805_2012Metric, symbol Device:C
- added C32: 10uF, Capacitor_SMD:C_0805_2012Metric, symbol Device:C
- added D6: 1N4148, Diode_THT:D_DO-35_SOD27_P7.62mm_Horizontal, symbol Diode:1N4148
- added D7: MBR0540, Diode_SMD:D_SOD-123, symbol Diode:MBR0540
- added R39, R41: 10k, Resistor_SMD:R_0805_2012Metric, symbol Device:R
- C14, C15, C16, C18, C21, C22, C23, C24, C25, C26: footprint (none) -> Capacitor_SMD:C_0805_2012Metric
- J5: footprint (none) -> Connector_FFC-FPC:Hirose_FH12-40S-0.5SH_1x40-1MP_P0.50mm_Horizontal
- L1: footprint (none) -> Inductor_SMD:L_0805_2012Metric
- R17, R18, R19, R20, R21, R22, R23, R24, R25, R26, R27, R28, R29, R30, R31, R32, R33, R34, R35, R36, R37, R38: footprint (none) -> Resistor_SMD:R_0805_2012Metric
- U1: footprint TPS61169DCKR:SOT65P210X110-5N -> TPS61169:SOT65P210X110-5N
- U3: footprint RA8875L3N:QFP50P1600X1600X160-100N -> ra8875:RA8875
- U7: footprint 74HC4050D:SO16 -> 74HC4050:SO16
Connections:
- net +24V: now also D7.1 (K)
- net +3V3: now also C27.1, C28.1, C29.1, C30.1, C31.1
- net +5V: now also C32.1, R41.1
- net GND: now also C27.2, C28.2, C29.2, C30.2, C31.2, C32.2, R39.2
- net LEDK: now also R39.1
- net PWM0: now also D6.1 (K)
- net at L1.2, U1.1 (SW): now also D7.2 (A)
- net at D5.2 (A), U1.4 (CTRL): now also D6.2 (A), R41.2
Other:
- moved on the sheet: C23, C24, C25, C26

Commit message: initial display pcb
Parts:
- removed D5: 1N4148, Diode_THT:D_DO-35_SOD27_P7.62mm_Horizontal, symbol Diode:1N4148
- added C33, C34: 0.1uF, Capacitor_SMD:C_0805_2012Metric, symbol Device:C
- R17, R18, R19, R20, R21, R22, R23, R24, R25, R26, R27, R28, R29, R30, R31, R32, R33, R34, R35, R36, R39, R41: footprint Resistor_SMD:R_0805_2012Metric -> Resistor_SMD:R_0402_1005Metric_Pad0.72x0.64mm_HandSolder
- Y1: footprint (none) -> Crystal:Crystal_SMD_3225-4Pin_3.2x2.5mm_HandSoldering
Connections:
- net +3V3 is gone; now on net +3.3V: C27.1, C28.1, C29.1, C30.1, C31.1, J5.4 (Pin_4)
- net PCLK is gone; now on net PIXCLK: R35.2
- net RA_MISO is gone; now on net MISO: U3.42 (SDO)
- net +3.3V: now also C33.1, C34.1
- net GND: now also C33.2, C34.2

Commit message: Updated Schematic
Parts:
- C31: value .01uF -> 0.1uF
Changed lines of the file:
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@@
 			)
 		)
-		(property "Value" ".01uF"
+		(property "Value" "0.1uF"
 			(at 311.15 52.0699 0)
 			(effects

Commit message: Updated Schematic
Parts:
- R17, R18, R19, R20, R21, R22, R23, R24, R25, R26, R27, R28, R29, R30, R31, R32, R33, R34, R35, R36, R39, R41: footprint Resistor_SMD:R_0402_1005Metric_Pad0.72x0.64mm_HandSolder -> Resistor_SMD:R_0805_2012Metric
Changed lines of the file:
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@@
 			)
 		)
-		(property "Footprint" "Resistor_SMD:R_0402_1005Metric_Pad0.72x0.64mm_HandSolder"
+		(property "Footprint" "Resistor_SMD:R_0805_2012Metric"
 			(at 482.6 77.978 90)
 			(effects
@@
 			)
 		)
-		(property "Footprint" "Resistor_SMD:R_0402_1005Metric_Pad0.72x0.64mm_HandSolder"
+		(property "Footprint" "Resistor_SMD:R_0805_2012Metric"
 			(at 482.6 85.598 90)
 			(effects
@@
 			)
 		)
-		(property "Footprint" "Resistor_SMD:R_0402_1005Metric_Pad0.72x0.64mm_HandSolder"
+		(property "Footprint" "Resistor_SMD:R_0805_2012Metric"
 			(at 482.6 70.358 90)
 			(effects
@@
 			)
 		)
-		(property "Footprint" "Resistor_SMD:R_0402_1005Metric_Pad0.72x0.64mm_HandSolder"
+		(property "Footprint" "Resistor_SMD:R_0805_2012Metric"
 			(at 482.6 75.438 90)
 			(effects
@@
 			)
 		)
-		(property "Footprint" "Resistor_SMD:R_0402_1005Metric_Pad0.72x0.64mm_HandSolder"
+		(property "Footprint" "Resistor_SMD:R_0805_2012Metric"
 			(at 482.6 90.678 90)
 			(effects
@@
 			)
 		)
-		(property "Footprint" "Resistor_SMD:R_0402_1005Metric_Pad0.72x0.64mm_HandSolder"
+		(property "Footprint" "Resistor_SMD:R_0805_2012Metric"
 			(at 482.6 72.898 90)
 			(effects
@@
 			)
 		)
-		(property "Footprint" "Resistor_SMD:R_0402_1005Metric_Pad0.72x0.64mm_HandSolder"
+		(property "Footprint" "Resistor_SMD:R_0805_2012Metric"
 			(at 482.6 83.058 90)
 			(effects
@@
 			)
 		)
-		(property "Footprint" "Resistor_SMD:R_0402_1005Metric_Pad0.72x0.64mm_HandSolder"
+		(property "Footprint" "Resistor_SMD:R_0805_2012Metric"
 			(at 482.6 108.458 90)
 			(effects
@@
 			)
 		)
-		(property "Footprint" "Resistor_SMD:R_0402_1005Metric_Pad0.72x0.64mm_HandSolder"
+		(property "Footprint" "Resistor_SMD:R_0805_2012Metric"
 			(at 482.6 105.918 90)
 			(effects
@@
 			)
 		)
-		(property "Footprint" "Resistor_SMD:R_0402_1005Metric_Pad0.72x0.64mm_HandSolder"
+		(property "Footprint" "Resistor_SMD:R_0805_2012Metric"
 			(at 482.6 98.298 90)
 			(effects
@@
 			)
 		)
-		(property "Footprint" "Resistor_SMD:R_0402_1005Metric_Pad0.72x0.64mm_HandSolder"
+		(property "Footprint" "Resistor_SMD:R_0805_2012Metric"
 			(at 482.6 110.998 90)
 			(effects
@@
 			)
 		)
-		(property "Footprint" "Resistor_SMD:R_0402_1005Metric_Pad0.72x0.64mm_HandSolder"
+		(property "Footprint" "Resistor_SMD:R_0805_2012Metric"
 			(at 482.6 88.138 90)
 			(effects
@@
 			)
 		)
-		(property "Footprint" "Resistor_SMD:R_0402_1005Metric_Pad0.72x0.64mm_HandSolder"
+		(property "Footprint" "Resistor_SMD:R_0805_2012Metric"
 			(at 482.6 116.078 90)
 			(effects
@@
 			)
 		)
-		(property "Footprint" "Resistor_SMD:R_0402_1005Metric_Pad0.72x0.64mm_HandSolder"
+		(property "Footprint" "Resistor_SMD:R_0805_2012Metric"
 			(at 482.6 67.818 90)
 			(effects
@@
 			)
 		)
-		(property "Footprint" "Resistor_SMD:R_0402_1005Metric_Pad0.72x0.64mm_HandSolder"
+		(property "Footprint" "Resistor_SMD:R_0805_2012Metric"
 			(at 482.6 103.378 90)
 			(effects
@@
 			)
 		)
-		(property "Footprint" "Resistor_SMD:R_0402_1005Metric_Pad0.72x0.64mm_HandSolder"
+		(property "Footprint" "Resistor_SMD:R_0805_2012Metric"
 			(at 64.262 54.61 90)
 			(effects
@@
 			)
 		)
-		(property "Footprint" "Resistor_SMD:R_0402_1005Metric_Pad0.72x0.64mm_HandSolder"
+		(property "Footprint" "Resistor_SMD:R_0805_2012Metric"
 			(at 482.6 80.518 90)
 			(effects
@@
 			)
 		)
-		(property "Footprint" "Resistor_SMD:R_0402_1005Metric_Pad0.72x0.64mm_HandSolder"
+		(property "Footprint" "Resistor_SMD:R_0805_2012Metric"
 			(at 482.6 93.218 90)
 			(effects
@@
 			)
 		)
-		(property "Footprint" "Resistor_SMD:R_0402_1005Metric_Pad0.72x0.64mm_HandSolder"
+		(property "Footprint" "Resistor_SMD:R_0805_2012Metric"
 			(at 143.002 64.77 90)
 			(effects
@@
 			)
 		)
-		(property "Footprint" "Resistor_SMD:R_0402_1005Metric_Pad0.72x0.64mm_HandSolder"
+		(property "Footprint" "Resistor_SMD:R_0805_2012Metric"
 			(at 482.6 95.758 90)
 			(effects
@@
 			)
 		)
-		(property "Footprint" "Resistor_SMD:R_0402_1005Metric_Pad0.72x0.64mm_HandSolder"
+		(property "Footprint" "Resistor_SMD:R_0805_2012Metric"
 			(at 482.6 100.838 90)
 			(effects
@@
 			)
 		)
-		(property "Footprint" "Resistor_SMD:R_0402_1005Metric_Pad0.72x0.64mm_HandSolder"
+		(property "Footprint" "Resistor_SMD:R_0805_2012Metric"
 			(at 482.6 113.538 90)
 			(effects

Commit message: re-layout of display subsystem
Parts:
- L1: footprint Inductor_SMD:L_0805_2012Metric -> Boost_Inductor:IND_TAIYO_NR5040_TAY
Changed lines of the file:
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@@
 			)
 		)
-		(property "Footprint" "Inductor_SMD:L_0805_2012Metric"
+		(property "Footprint" "Boost_Inductor:IND_TAIYO_NR5040_TAY"
 			(at 99.06 36.83 0)
 			(effects
