File: hall_effect.kicad_sch (KiCad schematic)
At the start: 30 parts, among them J10 Conn_01x01_Pin, J11 Conn_01x01_Pin, J12 Conn_01x01_Pin, J2 Conn_01x03_Pin, J8 Conn_01x03_Pin, J9 Conn_01x01_Pin, U12 OPA196xDGK, U13 OPA196xDGK, U2 OPA196xDGK, U4 OPA196xDGK

Commit message: Fixed labels and added datasheets
Changed lines of the file:
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@@
+	(wire
+		(pts
+			(xy 158.75 97.79) (xy 184.15 97.79)
+		)
+		(stroke
+			(width 0)
+			(type default)
+		)
+	)
 	(wire
 		(pts
@@
 	(wire
 		(pts
-			(xy 172.72 71.12) (xy 173.99 71.12)
+			(xy 172.72 71.12) (xy 182.88 71.12)
 		)
 		(stroke
@@
 	(wire
 		(pts
+			(xy 160.02 102.87) (xy 185.42 102.87)
+		)
+		(stroke
+			(width 0)
+			(type default)
+		)
+	)
+	(wire
+		(pts
 			(xy 91.44 130.81) (xy 93.98 130.81)
 		)
@@
 	(wire
 		(pts
-			(xy 168.91 102.87) (xy 185.42 102.87)
-		)
-		(stroke
-			(width 0)
-			(type default)
-		)
-	)
-	(wire
-		(pts
-			(xy 162.56 135.89) (xy 165.1 135.89)
+			(xy 162.56 135.89) (xy 172.72 135.89)
 		)
 		(stroke
@@
 		(pts
 			(xy 77.47 72.39) (xy 77.47 73.66)
-		)
-		(stroke
-			(width 0)
-			(type default)
-		)
-	)
-	(wire
-		(pts
-			(xy 167.64 97.79) (xy 184.15 97.79)
 		)
 		(stroke
@@
 		)
 	)
+	(label "ADC_IN1"
+		(at 158.75 97.79 0)
+		(effects
+			(font
+				(size 1.27 1.27)
+			)
+			(justify left bottom)
+		)
+	)
+	(label "ADC_IN2"
+		(at 172.72 135.89 180)
+		(effects
+			(font
+				(size 1.27 1.27)
+			)
+			(justify right bottom)
+		)
+	)
+	(label "ADC_IN2"
+		(at 160.02 102.87 0)
+		(effects
+			(font
+				(size 1.27 1.27)
+			)
+			(justify left bottom)
+		)
+	)
+	(label "ADC_IN1"
+		(at 182.88 71.12 180)
+		(effects
+			(font
+				(size 1.27 1.27)
+			)
+			(justify right bottom)
+		)
+	)
 	(label "VDDA"
 		(at 58.42 116.84 90)
@@
 		)
 	)
-	(global_label "ADC_IN2"
-		(shape input)
-		(at 168.91 102.87 180)
-		(fields_autoplaced yes)
-		(effects
-			(font
-				(size 1.27 1.27)
-			)
-			(justify right)
-		)
-		(property "Intersheetrefs" "${INTERSHEET_REFS}"
-			(at 158.1838 102.87 0)
-			(effects
-				(font
-					(size 1.27 1.27)
-				)
-				(justify right)
-				(hide yes)
-			)
-		)
-	)
-	(global_label "ADC_IN2"
-		(shape input)
-		(at 165.1 135.89 0)
-		(fields_autoplaced yes)
+	(hierarchical_label "ADC_IN2"
+		(shape output)
+		(at 185.42 102.87 0)
 		(effects
 			(font
@@
 			(justify left)
 		)
-		(property "Intersheetrefs" "${INTERSHEET_REFS}"
-			(at 175.8262 135.89 0)
-			(effects
-				(font
-					(size 1.27 1.27)
-				)
-				(justify left)
-				(hide yes)
-			)
-		)
-	)
-	(global_label "ADC_IN1"
-		(shape input)
-		(at 167.64 97.79 180)
-		(fields_autoplaced yes)
-		(effects
-			(font
-				(size 1.27 1.27)
-			)
-			(justify right)
-		)
-		(property "Intersheetrefs" "${INTERSHEET_REFS}"
-			(at 156.9138 97.79 0)
-			(effects
-				(font
-					(size 1.27 1.27)
-				)
-				(justify right)
-				(hide yes)
-			)
-		)
-	)
-	(global_label "ADC_IN1"
-		(shape input)
-		(at 173.99 71.12 0)
-		(fields_autoplaced yes)
-		(effects
-			(font
-				(size 1.27 1.27)
-			)
-			(justify left)
-		)
-		(property "Intersheetrefs" "${INTERSHEET_REFS}"
-			(at 184.7162 71.12 0)
-			(effects
-				(font
-					(size 1.27 1.27)
-				)
-				(justify left)
-				(hide yes)
-			)
-		)
-	)
-	(hierarchical_label "ADC_IN2"
-		(shape input)
-		(at 185.42 102.87 0)
-		(effects
-			(font
-				(size 1.27 1.27)
-			)
-			(justify left)
-		)
 	)
 	(hierarchical_label "ADC_IN1"
-		(shape input)
+		(shape output)
 		(at 184.15 97.79 0)
 		(effects
