File: senior_design.kicad_pcb (KiCad board)
At the start: 2 copper layers, 128.6 x 80.8 mm, 136 parts, among them J10 Conn_01x01_Pin, J11 Conn_01x01_Pin, J12 Conn_01x01_Pin, J13 Conn_ARM_JTAG_SWD_10, J2 Conn_01x03_Pin, J3 Conn_01x09_Socket, J4 USB_B_Micro, J5 Out_to_display, J6 AudioJack3, J7 SD_Card_Receptacle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

Commit message: fixed several issues from review
Connections:
- C36 pad 2: GND -> GNDA
- D8 pad 1: GND -> GNDA
- J6 pad S: GND -> GNDA
Routing:
- net GNDA: track 40.7 -> 47.5 mm, vias 15 -> 17
- net GND: track 223.0 -> 216.2 mm, vias 88 -> 86
Changed lines of the file:
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@@
 			(layers "F.Cu" "F.Mask" "F.Paste")
 			(roundrect_rratio 0.075)
-			(net 2 "GND")
+			(net 27 "GNDA")
 			(pinfunction "A1")
 			(pintype "passive")
@@
 			)
 		)
-		(property "Datasheet" "~"
+		(property "Datasheet" "https://www.raltron.com/webproducts/specs/CRYSTAL/RH100-8.000-10-1010-EXT-TR.pdf"
 			(at 0 0 0)
 			(layer "F.Fab")
@@
 			(size 2.8 2.2)
 			(layers "F.Cu" "F.Mask" "F.Paste")
-			(net 2 "GND")
+			(net 27 "GNDA")
 			(pintype "passive")
 		)
@@
 			(layers "B.Cu" "B.Mask" "B.Paste")
 			(roundrect_rratio 0.212766)
-			(net 2 "GND")
+			(net 27 "GNDA")
 			(pintype "passive")
 		)
@@
 	)
 	(segment
-		(start 139.7825 123.475)
-		(end 136.8375 123.475)
-		(width 0.2)
-		(layer "F.Cu")
-		(net 2)
-	)
-	(segment
 		(start 169.475 78.18)
 		(end 169.475 76.975)
@@
 	)
 	(segment
-		(start 157.7875 125.225)
-		(end 160.7625 125.225)
-		(width 0.2)
-		(layer "F.Cu")
-		(net 2)
-	)
-	(segment
 		(start 210.5 93.85)
 		(end 211.9 93.85)
@@
 	)
 	(segment
-		(start 136.8375 123.475)
-		(end 136.2125 124.1)
-		(width 0.2)
-		(layer "F.Cu")
-		(net 2)
-	)
-	(segment
 		(start 196.625 92)
 		(end 196.625 93.925)
@@
 	)
 	(via
-		(at 160.9875 125)
-		(size 0.64)
-		(drill 0.381)
-		(layers "F.Cu" "B.Cu")
-		(net 2)
-	)
-	(via
 		(at 222.15 82.5)
 		(size 0.64)
@@
 	)
 	(via
-		(at 136.2125 124.1)
-		(size 0.64)
-		(drill 0.381)
-		(layers "F.Cu" "B.Cu")
-		(net 2)
-	)
-	(via
 		(at 231.03 59.38)
 		(size 0.6)
@@
 	)
 	(segment
+		(start 139.7825 123.475)
+		(end 136.8375 123.475)
+		(width 0.2)
+		(layer "F.Cu")
+		(net 27)
+	)
+	(segment
 		(start 182.9625 87.3375)
 		(end 182.775 87.525)
@@
 	)
 	(segment
+		(start 157.7875 125.225)
+		(end 160.7625 125.225)
+		(width 0.2)
+		(layer "F.Cu")
+		(net 27)
+	)
+	(segment
 		(start 134.01 77.19)
 		(end 133.99 77.17)
@@
 	)
 	(segment
+		(start 136.8375 123.475)
+		(end 136.2125 124.1)
+		(width 0.2)
+		(layer "F.Cu")
+		(net 27)
+	)
+	(segment
 		(start 145.58 94.83)
 		(end 145.5 94.75)
@@
 	)
 	(via
+		(at 160.9875 125)
+		(size 0.64)
+		(drill 0.381)
+		(layers "F.Cu" "B.Cu")
+		(net 27)
+	)
+	(via
 		(at 140.45 92.95)
 		(size 0.64)
@@
 	)
 	(via
+		(at 136.2125 124.1)
+		(size 0.64)
+		(drill 0.381)
+		(layers "F.Cu" "B.Cu")
+		(net 27)
+	)
+	(via
 		(at 130.475 96.025)
 		(size 0.64)
@@
 		(polygon
 			(pts
+				(xy 230.725 66.95) (xy 230.730132 61.225316) (xy 236.325 61.2) (xy 236.370569 66.946764)
+			)
+		)
+	)
+	(zone
+		(net 0)
+		(net_name "")
+		(layers "F.Cu" "B.Cu")
+		(hatch edge 0.5)
+		(connect_pads
+			(clearance 0)
+		)
+		(min_thickness 0.25)
+		(filled_areas_thickness no)
+		(keepout
+			(tracks allowed)
+			(vias allowed)
+			(pads allowed)
+			(copperpour not_allowed)
+			(footprints allowed)
+		)
+		(placement
+			(enabled no)
+			(sheetname "")
+		)
+		(fill
+			(thermal_gap 0.5)
+			(thermal_bridge_width 0.5)
+		)
+		(polygon
+			(pts
 				(xy 124.925 130.925) (xy 134.35 130.95) (xy 134.325 120.675) (xy 124.85 120.675)
 			)
@@
 		(polygon
 			(pts
+				(xy 166.125 111.725) (xy 187.375 111.55) (xy 187.525 116.9) (xy 165.9 117.75)
+			)
+		)
+	)
+	(zone
+		(net 0)
+		(net_name "")
+		(layers "F.Cu" "B.Cu")
+		(hatch edge 0.5)
+		(connect_pads
+			(clearance 0)
+		)
+		(min_thickness 0.25)
+		(filled_areas_thickness no)
+		(keepout
+			(tracks allowed)
+			(vias allowed)
+			(pads allowed)
+			(copperpour not_allowed)
+			(footprints allowed)
+		)
+		(placement
+			(enabled no)
+			(sheetname "")
+		)
+		(fill
+			(thermal_gap 0.5)
+			(thermal_bridge_width 0.5)
+		)
+		(polygon
+			(pts
 				(xy 211.8 75.6) (xy 205.67 75.585) (xy 205.82 80.335) (xy 205.025 80.35) (xy 205.025 82.55) (xy 207.325 82.6)
 				(xy 207.375 85.25) (xy 209.625 87.95) (xy 210.15 85.15) (xy 211.041935 83.100605) (xy 213.05 82.95)
@@
 			(pts
 				(xy 123.625 71.5) (xy 132.4 72.05) (xy 138.75 73.2) (xy 154.425 74.225) (xy 164.475 82.3) (xy 172.175 82.975)
-				(xy 175.9 83.375) (xy 180.9 90.375) (xy 177.65 94.625) (xy 168.475 102.3) (xy 153.375 107.5) (xy 146.4 108.925)
-				(xy 123.85 113.025)
+				(xy 175.9 83.375) (xy 180.9 90.375) (xy 177.65 94.625) (xy 168.597726 102.197338) (xy 158.3 113.475)
+				(xy 162.049456 126.195373) (xy 151.1 130.55) (xy 140.075 128.925) (xy 123.85 113.025)
 			)
 		)
